File: hardware/gps-rx.kicad_sch (KiCad schematic)
At the start: 7 parts, among them J1 Conn_Coaxial_Small, U1 ICE40UP5K-SG48I, U5 MAX2769C

Commit message: new project specific library
Parts:
- removed FL1: SAFFB1G56KB0F0A, Filter:Filter_1109-5_1.1x0.9mm, symbol Filter:SAFFB1G56KB0F0A
- removed U5: MAX2769C, Package_DFN_QFN:TQFN-28-1EP_5x5mm_P0.5mm_EP3.25x3.25mm, symbol RF:MAX2769C
- added FL2: SAFFB1G56KB0F0A, Filter:Filter_1109-5_1.1x0.9mm, symbol gps-rx-lib:SAFFB1G56KB0F0A
- added U2: MAX2769C, Package_DFN_QFN:TQFN-28-1EP_5x5mm_P0.5mm_EP3.25x3.25mm, symbol gps-rx-lib:MAX2769C
Connections:
- net GND: now also FL2.2, FL2.3, FL2.5, U2.29 (EP)
- net at C2.2: now also FL2.4
- net at C1.1: now also FL2.1
Changed lines of the file:
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@@
+	)
+	(symbol
+		(lib_id "gps-rx-lib:SAFFB1G56KB0F0A")
+		(at 147.32 176.53 0)
+		(unit 1)
+		(body_style 1)
+		(exclude_from_sim no)
+		(in_bom yes)
+		(on_board yes)
+		(in_pos_files yes)
+		(dnp no)
+		(fields_autoplaced yes)
+		(property "Reference" "FL2"
+			(at 147.32 166.37 0)
+			(show_name no)
+			(do_not_autoplace no)
+			(effects
+				(font
+					(size 1.27 1.27)
+				)
+			)
+		)
+		(property "Value" "SAFFB1G56KB0F0A"
+			(at 147.32 168.91 0)
+			(show_name no)
+			(do_not_autoplace no)
+			(effects
+				(font
+					(size 1.27 1.27)
+				)
+			)
+		)
+		(property "Footprint" "Filter:Filter_1109-5_1.1x0.9mm"
+			(at 147.32 176.53 0)
+			(hide yes)
+			(show_name no)
+			(do_not_autoplace no)
+			(effects
+				(font
+					(size 1.27 1.27)
+				)
+			)
+		)
+		(property "Datasheet" "https://www.lcsc.com/datasheet/C91647.pdf"
+			(at 145.542 175.768 0)
+			(hide yes)
+			(show_name no)
+			(do_not_autoplace no)
+			(effects
+				(font
+					(size 1.27 1.27)
+				)
+			)
+		)
+		(property "Description" "Murata 1575.42/1602MHz SAW filter, SMD 1109"
+			(at 147.32 176.53 0)
+			(hide yes)
+			(show_name no)
+			(do_not_autoplace no)
+			(effects
+				(font
+					(size 1.27 1.27)
+				)
+			)
+		)
+		(pin "1"
+		)
+		(pin "4"
+		)
+		(pin "3"
+		)
+		(pin "5"
+		)
+		(pin "2"
+		)
+		(instances
+			(project "gps-rx"
+				(path "/da1c0f38-a7a5-4501-8e23-326add1cbb76"
+					(reference "FL2")
+					(unit 1)
+				)
+			)
+		)
 	)
 	(symbol
@@
 	)
 	(symbol
+		(lib_id "gps-rx-lib:MAX2769C")
+		(at 217.17 185.42 0)
+		(unit 1)
+		(body_style 1)
+		(exclude_from_sim no)
+		(in_bom yes)
+		(on_board yes)
+		(in_pos_files yes)
+		(dnp no)
+		(fields_autoplaced yes)
+		(property "Reference" "U2"
+			(at 219.3133 209.55 0)
+			(show_name no)
+			(do_not_autoplace no)
+			(effects
+				(font
+					(size 1.27 1.27)
+				)
+				(justify left)
+			)
+		)
+		(property "Value" "MAX2769C"
+			(at 219.3133 212.09 0)
+			(show_name no)
+			(do_not_autoplace no)
+			(effects
+				(font
+					(size 1.27 1.27)
+				)
+				(justify left)
+			)
+		)
+		(property "Footprint" "Package_DFN_QFN:TQFN-28-1EP_5x5mm_P0.5mm_EP3.25x3.25mm"
+			(at 217.17 185.42 0)
+			(hide yes)
+			(show_name no)
+			(do_not_autoplace no)
+			(effects
+				(font
+					(size 1.27 1.27)
+				)
+			)
+		)
+		(property "Datasheet" "https://www.analog.com/media/en/technical-documentation/data-sheets/max2769.pdf"
+			(at 217.17 185.42 0)
+			(hide yes)
+			(show_name no)
+			(do_not_autoplace no)
+			(effects
+				(font
+					(size 1.27 1.27)
+				)
+			)
+		)
+		(property "Description" "1.55GHz~1.61GHz 1.57542GHz 2.7V~3.3V QFN-28-EP(5x5) RF Transceiver ICs GPS RoHS"
+			(at 217.17 185.42 0)
+			(hide yes)
+			(show_name no)
+			(do_not_autoplace no)
+			(effects
+				(font
+					(size 1.27 1.27)
+				)
+			)
+		)
+		(pin "1"
+		)
+		(pin "11"
+		)
+		(pin "17"
+		)
+		(pin "28"
+		)
+		(pin "12"
+		)
+		(pin "14"
+		)
+		(pin "29"
+		)
+		(pin "7"
+		)
+		(pin "8"
+		)
+		(pin "24"
+		)
+		(pin "23"
+		)
+		(pin "15"
+		)
+		(pin "26"
+		)
+		(pin "2"
+		)
+		(pin "21"
+		)
+		(pin "3"
+		)
+		(pin "4"
+		)
+		(pin "9"
+		)
+		(pin "19"
+		)
+		(pin "10"
+		)
+		(pin "6"
+		)
+		(pin "25"
+		)
+		(pin "16"
+		)
+		(pin "27"
+		)
+		(pin "13"
+		)
+		(pin "22"
+		)
+		(pin "18"
+		)
+		(pin "20"
+		)
+		(pin "5"
+		)
+		(instances
+			(project "gps-rx"
+				(path "/da1c0f38-a7a5-4501-8e23-326add1cbb76"
+					(reference "U2")
+					(unit 1)
+				)
+			)
+		)
+	)
+	(symbol
 		(lib_id "FPGA_Lattice:ICE40UP5K-SG48ITR")
 		(at 151.13 76.2 0)
@@
 					(reference "U1")
 					(unit 3)
-				)
-			)
-		)
-	)
-	(symbol
-		(lib_id "Filter:SAFFB1G56KB0F0A")
-		(at 147.32 176.53 0)
-		(unit 1)
-		(body_style 1)
-		(exclude_from_sim no)
-		(in_bom yes)
-		(on_board yes)
-		(in_pos_files yes)
-		(dnp no)
-		(fields_autoplaced yes)
-		(property "Reference" "FL1"
-			(at 147.32 166.37 0)
-			(show_name no)
-			(do_not_autoplace no)
-			(effects
-				(font
-					(size 1.27 1.27)
-				)
-			)
-		)
-		(property "Value" "SAFFB1G56KB0F0A"
-			(at 147.32 168.91 0)
-			(show_name no)
-			(do_not_autoplace no)
-			(effects
-				(font
-					(size 1.27 1.27)
-				)
-			)
-		)
-		(property "Footprint" "Filter:Filter_1109-5_1.1x0.9mm"
-			(at 147.32 176.53 0)
-			(hide yes)
-			(show_name no)
-			(do_not_autoplace no)
-			(effects
-				(font
-					(size 1.27 1.27)
-				)
-			)
-		)
-		(property "Datasheet" "https://www.murata.com/~/media/webrenewal/support/library/catalog/products/filter/rf/p73e.ashx?la=en"
-			(at 145.542 175.768 0)
-			(hide yes)
-			(show_name no)
-			(do_not_autoplace no)
-			(effects
-				(font
-					(size 1.27 1.27)
-				)
-			)
-		)
-		(property "Description" "Murata 1575.42/1602MHz SAW filter, SMD 1109"
-			(at 147.32 176.53 0)
-			(hide yes)
-			(show_name no)
-			(do_not_autoplace no)
-			(effects
-				(font
-					(size 1.27 1.27)
-				)
-			)
-		)
-		(pin "5"
-		)
-		(pin "2"
-		)
-		(pin "3"
-		)
-		(pin "4"
-		)
-		(pin "1"
-		)
-		(instances
-			(project "gps-rx"
-				(path "/da1c0f38-a7a5-4501-8e23-326add1cbb76"
-					(reference "FL1")
-					(unit 1)
 				)
 			)
@@
 					(unit 1)
 				)
-			)
-		)
-	)
-	(symbol
-		(lib_id "RF:MAX2769C")
-		(at 217.17 185.42 0)
-		(unit 1)
-		(body_style 1)
-		(exclude_from_sim no)
-		(in_bom yes)
-		(on_board yes)
-		(in_pos_files yes)
-		(dnp no)
-		(fields_autoplaced yes)
-		(property "Reference" "U5"
-			(at 219.3133 209.55 0)
-			(show_name no)
-			(do_not_autoplace no)
-			(effects
-				(font
-					(size 1.27 1.27)
-				)
-				(justify left)
-			)
-		)
-		(property "Value" "MAX2769C"
-			(at 219.3133 212.09 0)
-			(show_name no)
-			(do_not_autoplace no)
-			(effects
-				(font
-					(size 1.27 1.27)
-				)
-				(justify left)
-			)
-		)
-		(property "Footprint" "Package_DFN_QFN:TQFN-28-1EP_5x5mm_P0.5mm_EP3.25x3.25mm"
-			(at 217.17 185.42 0)
-			(hide yes)
-			(show_name no)
-			(do_not_autoplace no)
-			(effects
-				(font
-					(size 1.27 1.27)
-				)
-			)
-		)
-		(property "Datasheet" "https://www.analog.com/media/en/technical-documentation/data-sheets/max2769.pdf"
-			(at 217.424 218.948 0)
-			(hide yes)
-			(show_name no)
-			(do_not_autoplace no)
-			(effects
-				(font
-					(size 1.27 1.27)
-				)
-			)
-		)
-		(property "Description" "1.55GHz~1.61GHz 1.57542GHz 2.7V~3.3V QFN-28-EP(5x5) RF Transceiver ICs GPS RoHS"
-			(at 217.424 218.948 0)
-			(hide yes)
-			(show_name no)
-			(do_not_autoplace no)
-			(effects
-				(font
-					(size 1.27 1.27)
-				)
-			)
-		)
-		(pin "6"
-		)
-		(pin "11"
-		)
-		(pin "19"
-		)
-		(pin "20"
-		)
-		(pin "13"
-		)
-		(pin "2"
-		)
-		(pin "27"
-		)
-		(pin "17"
-		)
-		(pin "25"
-		)
-		(pin "28"
-		)
-		(pin "23"
-		)
-		(pin "4"
-		)
-		(pin "16"
-		)
-		(pin "18"
-		)
-		(pin "24"
-		)
-		(pin "1"
-		)
-		(pin "5"
-		)
-		(pin "15"
-		)
-		(pin "10"
-		)
-		(pin "3"
-		)
-		(pin "7"
-		)
-		(pin "8"
-		)
-		(pin "9"
-		)
-		(pin "12"
-		)
-		(pin "14"
-		)
-		(pin "21"
-		)
-		(pin "22"
-		)
-		(pin "26"
-		)
-		(pin "29"
-		)
-		(instances
-			(project "gps-rx"
-				(path "/da1c0f38-a7a5-4501-8e23-326add1cbb76"
-					(reference "U5")
-					(unit 1)
-				)
