File: hardware/gps-rx.kicad_sch (KiCad schematic)
At the start: 7 parts, among them J1 Conn_Coaxial_Small, U1 ICE40UP5K-SG48I, U2 MAX2769C

Commit message: new stuff
Parts:
- added C1, C10, C12, C13, C14, C15, C16, C17, C18, C2, C4, C8: 100n, Capacitor_SMD:C_0402_1005Metric, symbol Device:C_Small
- added C11, C9: 100p, Capacitor_SMD:C_0402_1005Metric, symbol Device:C_Small
- added C19: 27p, Capacitor_SMD:C_0402_1005Metric, symbol Device:C_Small
- added C20, C7: 470p, Capacitor_SMD:C_0402_1005Metric, symbol Device:C_Small
- added C21, C22: 10u, Capacitor_SMD:C_0805_2012Metric, symbol Device:C
- added C6: 10n, Capacitor_SMD:C_0402_1005Metric, symbol Device:C_Small
- added D1: LED, LED_SMD:LED_0402_1005Metric, symbol Device:LED
- added H1, H2: MountingHole, MountingHole:MountingHole_2.2mm_M2, symbol Mechanical:MountingHole
- added J1: Conn_01x04_Pin, Connector_PinHeader_2.54mm:PinHeader_1x04_P2.54mm_Vertical, symbol Connector:Conn_01x04_Pin
- added L2: L, Inductor_SMD:L_0603_1608Metric, symbol Device:L
- added R1, R2, R5, R6: 10k, Resistor_SMD:R_0402_1005Metric, symbol Device:R_Small
- added R3: 220R, Resistor_SMD:R_0402_1005Metric, symbol Device:R_Small
- added R4: 20k, Resistor_SMD:R_0402_1005Metric, symbol Device:R_Small
- added TP1, TP10, TP2, TP3, TP4, TP5, TP6, TP7, TP8, TP9: TestPoint, TestPoint:TestPoint_Pad_D1.0mm, symbol Connector:TestPoint
- added U4: PAM2305CGF120, Package_DFN_QFN:DFN-6-1EP_2x2mm_P0.65mm_EP1x1.6mm, symbol Regulator_Switching:PAM2305CGF120
- added U5: W25Q16JVUXIQ, Package_SON:Winbond_USON-8-1EP_3x2mm_P0.5mm_EP0.2x1.6mm, symbol Memory_Flash:W25Q16JVSS
- added Y1: 1XXB16368MBA, Crystal:Crystal_SMD_2520-4Pin_2.5x2.0mm, symbol Oscillator:ECS-2520MV-xxx-xx
- C3: renamed from C1; value C_Small -> 470p; footprint (none) -> Capacitor_SMD:C_0402_1005Metric
- C5: renamed from C2; value C_Small -> 470p; footprint (none) -> Capacitor_SMD:C_0402_1005Metric
- J2: renamed from J1; footprint (none) -> Connector_Coaxial:U.FL_Molex_MCRF_73412-0110_Vertical
- L1: value L -> 27n; footprint (none) -> Inductor_SMD:L_0402_1005Metric
- renumbered FL2 to FL1, U1 to U2, U2 to U3
Connections:
- net MIXER_LO_IN is gone; now on net ~{CS}: U2.45 (IOB_5b)
- net ~{LNA_SHDN} is gone; now on net ANTFLAG: U2.3 (IOB_9b)
- net +3V3: now also U2.1 (VCCIO_2), U2.22 (SPI_VCCIO1), U2.24 (VPP_2V5), U2.33 (VCCIO_0), U3.11 (VCCVCO), U3.13 (VCCCP), U3.14 (VCCD), U3.19 (VCCADC), U3.23 (VCCIF), U3.4 (VCCRF), C1.1, C10.1, C11.1, C13.1, C15.1, C16.1, C17.1, C18.1, C2.1, C21.1, C4.1, C8.1, C9.1, J1.1 (Pin_1), R1.2, R2.2, R5.2, R6.2, TP8.1, U4.2 (EN), U4.3 (Vin), U5.8 (VCC), Y1.4 (VDD); no longer L1.1
- net GND: now also U2.49 (GND), C1.2, C10.2, C11.2, C12.2, C13.2, C14.2, C15.2, C16.2, C17.2, C18.2, C19.2, C2.2, C20.2, C21.2, C22.2, C4.2, C8.2, C9.2, D1.1 (K), J1.4 (Pin_4), TP9.1, U4.5 (GND), U4.7 (PAD), U5.4 (GND), U5.9 (GND), Y1.1 (GND), Y1.2 (GND)
- net RX: now reaches U2.25 (IOT_36b)
- net RX: now also J1.3 (Pin_3)
- net TX: now reaches U2.26 (IOT_39a)
- net TX: now also J1.2 (Pin_2)
- net at C5.1: now also U3.25 (LNA2)
- net +1V2: now reaches U2.29 (VCCPLL)
- net +1V2: now also U2.30 (VCC), U2.5 (VCC), C12.1, C14.1, C22.1, L2.2, TP10.1, U4.6 (FB)
- net ANTFLAG: now reaches U3.1 (ANTFLAG)
- net ~{CS}: now reaches U3.10 (~{CS})
- net at U3.12 (CPOUT): now also C19.1, R4.1
- net at U3.15 (XTAL): now also C6.2
- net CLKOUT: now reaches U3.16 (CLKOUT)
- net CLKOUT: now also U2.20 (IOB_25b_G3), TP1.1
- net Q1: now reaches U3.17 (Q1)
- net Q1: now also U2.12 (IOB_22a)
- net Q0: now reaches U3.18 (Q0)
- net Q0: now also U2.11 (IOB_20a)
- net LNAOUT: now reaches U3.2 (LNAOUT)
- net LNAOUT: now also C7.1
- net I0: now reaches U3.20 (I0)
- net I0: now also U2.10 (IOB_18a)
- net I1: now reaches U3.21 (I1)
- net I1: now also U2.9 (IOB_16a)
- net ~{IDLE}: now reaches U3.24 (~{IDLE})
- net PGM: now reaches U3.26 (PGM)
- net PGM: now also U2.6 (IOB_13b)
- net ANTIBIAS: now reaches U3.3 (ANTIBIAS)
- net ANTIBIAS: now also L1.1
- net MIXIN: now reaches U3.5 (MIXIN)
- net MIXIN: now also C7.2
- net LD: now reaches U3.6 (LD)
- net LD: now also U2.2 (IOB_6a)
- net ~{SHDN}: now reaches U3.7 (~{SHDN})
- net ~{SHDN}: now also U2.4 (IOB_8a)
- net SDATA: now reaches U3.8 (SDATA)
- net SDATA: now also U2.47 (IOB_2a)
- net SCLK: now reaches U3.9 (SCLK)
- net SCLK: now also U2.46 (IOB_0a)
- net qSPI_~{RESET}: now reaches U2.13 (IOB_24a)
- net qSPI_~{RESET}: now also R6.1, U5.7 (~{HOLD}/~{RESET}/IO_{3})
- net qSPI_SO: now reaches U2.14 (IOB_32a_SPI_SO)
- net qSPI_SO: now also TP3.1, U5.5 (DI/IO_{0})
- net qSPI_CLK: now reaches U2.15 (IOB_34a_SPI_SCK)
- net qSPI_CLK: now also TP5.1, U5.6 (CLK)
- net qSPI_~{CS}: now reaches U2.16 (IOB_35b_SPI_SS)
- net qSPI_~{CS}: now also TP6.1, U5.1 (~{CS})
- net qSPI_SI: now reaches U2.17 (IOB_33b_SPI_SI)
- net qSPI_SI: now also TP4.1, U5.2 (DO/IO_{1})
- net qSPI_~{WP}: now reaches U2.18 (IOB_31b)
- net qSPI_~{WP}: now also R5.1, U5.3 (~{WP}/IO_{2})
- net CDONE: now reaches U2.7 (CDONE)
- net CDONE: now also R2.1, R3.2, TP7.1
- net ~{CRESET}: now reaches U2.8 (~{CRESET})
- net ~{CRESET}: now also R1.1, TP2.1
- new net: C20.1, R4.2
- new net: L2.1, U4.4 (SW)
- new net: D1.2 (A), R3.1
- new net XTAL: C6.1, Y1.3 (OUT)
- no-connect marks 0 -> 4
Other:
- note added: "CLKOUT Pin only to a Global buffer pin"
- note added: "TO Be added: 1. A programming interface to the FPGA. Figure out something that can be programmed via testpoints/pogo pins and then make it look like a commercial GPS module, just without COCOM limits"
- moved on the sheet: C3, C5, FL1, J2, L1, U2C, U2D, U3

Commit message: new PCB design
Parts:
- removed C1, C10, C16, C17: 100n, Capacitor_SMD:C_0402_1005Metric, symbol Device:C_Small
- removed C7: 470p, Capacitor_SMD:C_0402_1005Metric, symbol Device:C_Small
- removed R5: 10k, Resistor_SMD:R_0402_1005Metric, symbol Device:R_Small
- removed TP1, TP8, TP9: TestPoint, TestPoint:TestPoint_Pad_D1.0mm, symbol Connector:TestPoint
- added C23, C24: 470p, Capacitor_SMD:C_0402_1005Metric, symbol Device:C_Small
- added J2: Conn_Coaxial_Small, Connector_Coaxial:U.FL_Molex_MCRF_73412-0110_Vertical, symbol Connector:Conn_Coaxial_Small
- renumbered J2 to J1, J1 to J3
Connections:
- net ANTFLAG: now also U2.37 (IOT_45a_G1); no longer U2.3 (IOB_9b)
- net GND: now also J2.2 (Ext)
- net I0: no longer U2.10 (IOB_18a)
- net I1: no longer U2.9 (IOB_16a)
- net LD: no longer U2.2 (IOB_6a)
- net LNAOUT: now also C23.2
- net MIXIN: now also C24.1
- net PGM: now also U2.21 (IOB_23b); no longer U2.6 (IOB_13b)
- net Q0: no longer U2.11 (IOB_20a)
- net Q1: no longer U2.12 (IOB_22a)
- net RX: no longer U2.25 (IOT_36b)
- net SCLK: no longer U2.46 (IOB_0a)
- net SDATA: no longer U2.47 (IOB_2a)
- net TX: no longer U2.26 (IOT_39a)
- net ~{CS}: no longer U2.45 (IOB_5b)
- net ~{IDLE}: now also U2.19 (IOB_29b)
- net ~{SHDN}: no longer U2.4 (IOB_8a)
- net at FL1.1: now also C23.1; no longer C3.1
- net at FL1.4: now also C24.2; no longer C5.2
- net ACTIVE: now reaches U3.25 (LNA2)
- net ACTIVE: now also C3.1; no longer C5.1
- net PASSIVE: now reaches U3.27 (LNA1)
- net PASSIVE: now also C5.1
- new net: C5.2, J2.1 (In)
- no-connect marks 4 -> 3
Other:
- note added: "ADD 2ND U.FL CONNECTOR FOR PASSIVE ANTENNAE"
- moved on the sheet: C18, C3, C6, J1, L1, Y1

Commit message: PCB completed
Parts:
- C21, C22: footprint Capacitor_SMD:C_0805_2012Metric -> Capacitor_SMD:C_0603_1608Metric
- L2: value L -> 2.2u; footprint Inductor_SMD:L_0603_1608Metric -> Inductor_SMD:L_0402_1005Metric
- R3: value 220R -> 1k
Connections:
- net ANTFLAG: now also U2.43 (IOT_49a); no longer U2.37 (IOT_45a_G1)
- net CLKOUT: now also U2.37 (IOT_45a_G1); no longer U2.20 (IOB_25b_G3)
- net I0: now also U2.26 (IOT_39a)
- net I1: now also U2.25 (IOT_36b)
- net LD: now also U2.36 (IOT_48b)
- net Q0: now also U2.11 (IOB_20a)
- net Q1: now also U2.10 (IOB_18a)
- net RX: now also U2.35 (IOT_46b_G0)
- net SCLK: now also U2.42 (IOT_51a)
- net SDATA: now also U2.31 (IOT_42b)
- net TX: now also U2.32 (IOT_43a)
- net ~{CS}: now also U2.34 (IOT_44b)
- net ~{SHDN}: now also U2.38 (IOT_50b)
Other:
- moved on the sheet: R6
